File: hardware/simHIT/sinHIT.kicad_sch (KiCad schematic)
At the start: 14 parts, among them P1 USB_C_Plug_USB2.0, SW1 SW_Push, U1 ESP-12E, U2 XC6206PxxxMR, U3 CH340G

Commit message: primera versión en pdf
Parts:
- removed R5: R, symbol Device:R
- removed U3: CH340G, Package_SO:SOIC-16_3.9x9.9mm_P1.27mm, symbol Interface_USB:CH340G
- added D1: LED_KRGB, symbol Device:LED_KRGB
- added J1: IMU, symbol Connector:Conn_01x04_Socket
- added LD1: SPL_PL90, LED_THT:LED_D5.0mm, symbol Diode_Laser:SPL_PL90
- added R10, R7, R8, R9: R, symbol Device:R
- added U3: CH340C, Package_SO:SOIC-16_3.9x9.9mm_P1.27mm, symbol Interface_USB:CH340C
- added U4: PC817, Package_DIP:DIP-4_W7.62mm, symbol Isolator:PC817
- R1, R2, R3, R6: value R -> 10k
- R4: value R -> 480
Connections:
- net +3.3V: now also J1.1 (Pin_1), U3.16 (VCC), U3.4 (V3), U4.1
- net +5V: now also P1.A4 (VBUS), P1.A9 (VBUS), P1.B4 (VBUS), P1.B9 (VBUS), D1.1 (K), U4.4
- net GND: now also P1.A1 (GND), P1.A12 (GND), P1.B1 (GND), P1.B12 (GND), P1.S1 (SHIELD), J1.4 (Pin_4), LD1.1 (C), U3.1 (GND)
- net rx: now also U3.2 (TXD)
- net tx: now also U3.3 (RXD)
- net buzzer: now reaches U1.17 (GPIO2)
- net SDA: now reaches U1.19 (GPIO4)
- net SDA: now also J1.2 (Pin_2)
- net SCL: now reaches U1.20 (GPIO5)
- net SCL: now also J1.3 (Pin_3)
- net led_blue: now reaches U1.4 (GPIO16)
- net led_blue: now also R9.2
- net led_green: now reaches U1.5 (GPIO14)
- net led_green: now also R8.2
- net Laser: now reaches U1.6 (GPIO12)
- net Laser: now also LD1.2 (A), U4.3
- net led_red: now reaches U1.7 (GPIO13)
- net led_red: now also R7.2
- net D+: now reaches P1.A6 (D+)
- net D+: now also U3.5 (UD+)
- net D-: now reaches P1.A7 (D-)
- net D-: now also U3.6 (UD-)
- new net: D1.3 (GA), R8.1
- new net: D1.2 (RA), R7.1
- new net: D1.4 (BA), R9.1
- new net: R10.2, U4.2
- no-connect marks 0 -> 9
Other:
- company: (none) -> Universidad Austral de Chile
- title: (none) -> SIMHIT
- moved on the sheet: R4, R6, SW1
